Commit message: Force visualisation of laser scan

File: urdf/sick_tim.urdf.xacro (robot description, xacro)
@@ -3,5 +3,5 @@
   xmlns:interface="http://playerstage.sourceforge.net/gazebo/xmlschema/#interface"
   xmlns:sensor="http://playerstage.sourceforge.net/gazebo/xmlschema/#sensor"
-  xmlns:xacro="http://ros.org/wiki/xacro">
+  xmlns:xacro="http://www.ros.org/wiki/xacro">
   <xacro:macro name="sick_tim310" params="name ros_topic">
     <xacro:sick_tim name="${name}" ros_topic="${ros_topic}"
@@ -62,5 +62,5 @@
         <update_rate>${update_rate}</update_rate>
         <pose>0 0 0 0 0 0</pose>
-        <visualize>false</visualize>
+        <visualize>true</visualize>
         <ray>
           <scan>

File: urdf/sick_tim_56x.urdf.xacro (robot description, xacro)
@@ -3,5 +3,5 @@
   xmlns:interface="http://playerstage.sourceforge.net/gazebo/xmlschema/#interface"
   xmlns:sensor="http://playerstage.sourceforge.net/gazebo/xmlschema/#sensor"
-  xmlns:xacro="http://ros.org/wiki/xacro">
+  xmlns:xacro="http://www.ros.org/wiki/xacro">
   <xacro:macro name="sick_tim561" params="name ros_topic parent">
     <xacro:sick_tim name="${name}" ros_topic="${ros_topic}"
@@ -22,5 +22,5 @@
           <mesh filename="${mesh}" />
         </geometry>
-        <material name="blue" >
+        <material name="blue">
           <color rgba="0 0 1 1" />
         </material>
@@ -48,5 +48,5 @@
         <update_rate>${update_rate}</update_rate>
         <pose>0 0 0 0 0 0</pose>
-        <visualize>false</visualize>
+        <visualize>true</visualize>
         <ray>
           <scan>
